File: hardware/Wii-Bluetooth-Sensor-Bar.kicad_sch (KiCad schematic)
At the start: 13 parts, among them J1 LED_Left, J2 LED_Right, SW1 SW_Push, U1 J27H002, U2 LM1117-3.3

Commit message: Update schematic/PCB
Parts:
- removed C1: 0.1uF, Capacitor_SMD:C_0805_2012Metric_Pad1.18x1.45mm_HandSolder, symbol Device:C_Small
- removed F1: 500mA, Fuse:Fuse_0805_2012Metric_Pad1.15x1.40mm_HandSolder, symbol Device:Fuse_Small
- removed R1, R2: 5.1K, Resistor_SMD:R_0805_2012Metric_Pad1.20x1.40mm_HandSolder, symbol Device:R_Small_US
- removed R5: 10K, Resistor_SMD:R_0805_2012Metric_Pad1.20x1.40mm_HandSolder, symbol Device:R_Small_US
- added C101: 0.1uF, Capacitor_SMD:C_0805_2012Metric_Pad1.18x1.45mm_HandSolder, symbol Device:C_Small
- added D101: PWR_GOOD, LED_THT:LED_D3.0mm, symbol Device:LED
- added F101: 500mA, Fuse:Fuse_1206_3216Metric_Pad1.42x1.75mm_HandSolder, symbol Device:Fuse
- added H101, H102, H103, H104: M2.5, MountingHole:MountingHole_2.7mm_M2.5, symbol Mechanical:MountingHole
- added R101, R102: 5.1k, Resistor_SMD:R_0805_2012Metric_Pad1.20x1.40mm_HandSolder, symbol Device:R
- added R103: 220, Resistor_SMD:R_0805_2012Metric_Pad1.20x1.40mm_HandSolder, symbol Device:R
- added R104: 10k, Resistor_SMD:R_0805_2012Metric_Pad1.20x1.40mm_HandSolder, symbol Device:R
- SW101: renamed from SW1; value SW_Push -> SYNC
- U101: renamed from U1; symbol Wii Bluetooth Module:J27H002 -> Foxconn:J27H002
- USB101: renamed from USB1; footprint Amphenol:USB_C_Receptacle_Amphenol_C12402012 -> Amphenol:GSB1C211110DS1HR
- renumbered C2 to C102, J1 to J101, J2 to J102, U2 to U102, USB2 to USB102
Connections:
- net +3V3: now also D101.2 (A)
- net +5V: now also U102.3 (VI), C101.1, F101.2; no longer USB101.A4 (VBUS), USB101.A9 (VBUS), USB101.B4 (VBUS), USB101.B9 (VBUS)
- net GND: now also C101.2, R101.1, R102.2, R103.2, R104.2
- net at SW101.2, U101.12 (SYNC): now also R104.1
- net at USB101.A5 (CC1): now also R102.1
- net at USB101.B5 (CC2): now also R101.2
- new net: D101.1 (K), R103.1
- new net VBUS: F101.1, USB101.A4 (VBUS), USB101.A9 (VBUS), USB101.B4 (VBUS), USB101.B9 (VBUS)
Other:
- note added: "3.3V REGULATOR"
- note added: "IR LED POWER PASSTHROUGH"
- note added: "USB POWER PASSTHROUGH"
- note added: "USB-C POWER/DATA CONNECTOR AND BLUETOOTH MODULE"
- note removed: "3.3V regulator"
- note removed: "IR LEDs"
- note removed: "USB passthrough for external sensor bar"
- note removed: "USB-C connector and Wii Bluetooth module"
- moved on the sheet: C102, J101, J102, SW101, U101, U102, USB101, USB102
